File: blinkie_pcb.kicad_sch (KiCad schematic)
At the start: 0 parts

Commit message: finished schematic
Parts:
- added C1: 1uF, symbol Device:C
- added C2: 0.01 UF, symbol Device:C
- added D1, D10, D2, D3, D4, D5, D6, D7, D8, D9: LED, symbol Device:LED
- added J1: Conn_01x01_Socket, symbol Connector:Conn_01x01_Socket
- added J2: Conn_01x02_Socket, symbol Connector:Conn_01x02_Socket
- added R1: R, symbol Device:R
- added R2: 470, symbol Device:R
- added RV1: R_Potentiometer, symbol Device:R_Potentiometer
- added U1: NE555P, Package_DIP:DIP-8_W7.62mm, symbol Timer:NE555P
- added U2: 4017, symbol 4xxx:4017
Connections:
- new net: C2.1, U1.5 (CONT)
- new net: R1.2, RV1.1, RV1.2, U1.7 (DISCH)
- new net: D1.1 (K), D10.1 (K), D2.1 (K), D3.1 (K), D4.1 (K), D5.1 (K), D6.1 (K), D7.1 (K), D8.1 (K), D9.1 (K), R2.1
- new net: D10.2 (A), U2.3 (Q0)
- new net: D5.2 (A), U2.5 (Q6)
- new net: D3.2 (A), U2.4 (Q2)
- new net: D8.2 (A), U2.2 (Q1)
- new net: D4.2 (A), U2.7 (Q3)
- new net: D7.2 (A), U2.9 (Q8)
- new net: D9.2 (A), U2.11 (Q9)
- new net: D6.2 (A), U2.6 (Q7)
- new net: D1.2 (A), U2.1 (Q5)
- new net: D2.2 (A), U2.10 (Q4)
- new net +5V: J2.1 (Pin_1), R1.1, U1.4 (~{RST}), U1.8 (VCC)
- new net GND: C1.1, C2.2, J2.2 (Pin_2), R2.2, U1.1 (GND), U2.13 (CKEN), U2.15 (Reset), U2.8 (VSS)
- new net OUT: J1.1 (Pin_1), U1.3 (OUT), U2.14 (CLK)
- new net TR: C1.2, RV1.3, U1.2 (TRIG), U1.6 (THRES)
- no-connect marks 0 -> 2

Commit message: DONEDONEDONEONDOIENE FINALLYYYY MY BACK HURTS
Parts:
- C1: footprint (none) -> Capacitor_THT:CP_Radial_D5.0mm_P2.00mm
- C2: footprint (none) -> Capacitor_THT:C_Disc_D7.5mm_W2.5mm_P5.00mm
- D1, D10, D2, D3, D4, D5, D6, D7, D8, D9: footprint (none) -> LED_THT:LED_D3.0mm
- J1: footprint (none) -> Connector_PinHeader_2.54mm:PinHeader_1x01_P2.54mm_Vertical
- J2: footprint (none) -> Connector_PinHeader_2.54mm:PinHeader_1x02_P2.54mm_Vertical
- R1, R2: footprint (none) -> Resistor_THT:R_Axial_DIN0207_L6.3mm_D2.5mm_P7.62mm_Horizontal
- RV1: footprint (none) -> Potentiometer_THT:Potentiometer_Vishay_T93YA_Vertical
- U2: footprint (none) -> imported:CD4017BE
Changed lines of the file:
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@@
 			)
 		)
-		(property "Footprint" ""
+		(property "Footprint" "LED_THT:LED_D3.0mm"
 			(at 215.9 58.42 0)
 			(effects
@@
 			)
 		)
-		(property "Footprint" ""
+		(property "Footprint" "Resistor_THT:R_Axial_DIN0207_L6.3mm_D2.5mm_P7.62mm_Horizontal"
 			(at 226.822 99.06 90)
 			(effects
@@
 			)
 		)
-		(property "Footprint" ""
+		(property "Footprint" "LED_THT:LED_D3.0mm"
 			(at 215.9 81.28 0)
 			(effects
@@
 			)
 		)
-		(property "Footprint" ""
+		(property "Footprint" "Capacitor_THT:C_Disc_D7.5mm_W2.5mm_P5.00mm"
 			(at 120.65 71.4248 0)
 			(effects
@@
 			)
 		)
-		(property "Footprint" ""
+		(property "Footprint" "LED_THT:LED_D3.0mm"
 			(at 215.9 66.04 0)
 			(effects
@@
 			)
 		)
-		(property "Footprint" ""
+		(property "Footprint" "LED_THT:LED_D3.0mm"
 			(at 215.9 62.23 0)
 			(effects
@@
 			)
 		)
-		(property "Footprint" ""
+		(property "Footprint" "LED_THT:LED_D3.0mm"
 			(at 215.9 69.85 0)
 			(effects
@@
 			)
 		)
-		(property "Footprint" ""
+		(property "Footprint" "Connector_PinHeader_2.54mm:PinHeader_1x01_P2.54mm_Vertical"
 			(at 63.5 29.21 0)
 			(effects
@@
 			)
 		)
-		(property "Footprint" ""
+		(property "Footprint" "Connector_PinHeader_2.54mm:PinHeader_1x02_P2.54mm_Vertical"
 			(at 34.29 30.48 0)
 			(effects
@@
 			)
 		)
-		(property "Footprint" ""
+		(property "Footprint" "LED_THT:LED_D3.0mm"
 			(at 215.9 88.9 0)
 			(effects
@@
 			)
 		)
-		(property "Footprint" ""
+		(property "Footprint" "Potentiometer_THT:Potentiometer_Vishay_T93YA_Vertical"
 			(at 80.01 92.71 0)
 			(effects
@@
 			)
 		)
-		(property "Footprint" ""
+		(property "Footprint" "Capacitor_THT:CP_Radial_D5.0mm_P2.00mm"
 			(at 83.82 103.1748 0)
 			(effects
@@
 			)
 		)
-		(property "Footprint" ""
+		(property "Footprint" "Resistor_THT:R_Axial_DIN0207_L6.3mm_D2.5mm_P7.62mm_Horizontal"
 			(at 78.232 82.55 90)
 			(effects
@@
 			)
 		)
-		(property "Footprint" ""
+		(property "Footprint" "LED_THT:LED_D3.0mm"
 			(at 215.9 92.71 0)
 			(effects
@@
 			)
 		)
-		(property "Footprint" ""
+		(property "Footprint" "LED_THT:LED_D3.0mm"
 			(at 215.9 85.09 0)
 			(effects
@@
 			)
 		)
-		(property "Footprint" ""
+		(property "Footprint" "LED_THT:LED_D3.0mm"
 			(at 215.9 77.47 0)
 			(effects
@@
 			)
 		)
-		(property "Footprint" ""
+		(property "Footprint" "LED_THT:LED_D3.0mm"
 			(at 215.9 73.66 0)
 			(effects
@@
 			)
 		)
-		(property "Footprint" ""
+		(property "Footprint" "imported:CD4017BE"
 			(at 184.15 77.47 0)
 			(effects
